Commit message: end effector added

File: config/ruka_gz.ros2_control.xacro (robot description, xacro)
@@ -37,4 +37,14 @@
                 <state_interface name="velocity"/>
             </joint>
+            <joint name="link_hand_cyl__first_fin">
+                <command_interface name="position"/>
+                <state_interface name="position"/>
+                <state_interface name="velocity"/>
+            </joint>
+            <joint name="link_hand_cyl__second_fin">
+                <command_interface name="position"/>
+                <state_interface name="position"/>
+                <state_interface name="velocity"/>
+            </joint>
       </ros2_control>
         <gazebo>

File: config/ruka_gz.urdf (robot description, URDF)
Before this commit: robot ruka_gz, 13 links, 12 joints
Links:
- added link first_fin, mass 0.01; collision mesh filename=file://$(find ruka_gz)/config/mesh/finger50mm-S.stl; visual mesh filename=file://$(find ruka_gz)/config/mesh/finger50mm-S.stl
- added link link_hand_cyl, mass 0.01; collision cylinder length=0.01 radius=0.010; visual mesh filename=file://$(find ruka_gz)/config/mesh/gripper4310.stl
- added link second_fin, mass 0.01; collision mesh filename=file://$(find ruka_gz)/config/mesh/finger50mm-S-1.stl; visual mesh filename=file://$(find ruka_gz)/config/mesh/finger50mm-S-1.stl
Joints:
- added joint link_06__link_hand_cyl: type fixed, parent link_06, child link_hand_cyl, origin xyz=0 0 0 rpy=0 0 0
- added joint link_hand_cyl__first_fin: type prismatic, parent link_hand_cyl, child first_fin, origin xyz=0 0.005 0.0642 rpy=1.57 0 3.14, axis 0 0 1, limit lower=0.0 upper=0.01 effort=20 velocity=0.2
- added joint link_hand_cyl__second_fin: type prismatic, parent link_hand_cyl, child second_fin, origin xyz=0 -0.005 0.0642 rpy=1.57 0 0, axis 0 0 1, limit lower=0.0 upper=0.01 effort=20 velocity=0.2

File: config/ruka_gz.urdf.xacro (robot description, xacro)
@@ -5,4 +5,5 @@
     <!-- Import ruka_hand urdf file -->
     <xacro:include filename="$(find ruka_gz)/config/ruka_gz.urdf" />
+    <!-- <xacro:include filename="$(find ruka_gz)/config/ruka_gz_hand.ros2_control.xacro" /> -->
     <!-- Import control_xacro -->
     <xacro:include filename="$(find ruka_gz)/config/ruka_gz.ros2_control.xacro" />
