Commit message: ros2 param set /move_group use_sim_time true

File: config/ruka_gz.urdf (robot description, URDF)
Before this commit: robot ruka_gz, 8 links, 7 joints
Links:
- added link link_01_red; collision box size=0.08 0.028 0.135; collision box size=0.08 0.028 0.135
- added link link_02_red; collision box size=0.076 0.198 0.025; collision box size=0.076 0.198 0.025
- added link link_03_red; collision box size=0.120 0.020 0.08; collision box size=0.120 0.020 0.08
- added link link_04_red; collision box size=0.18 0.020 0.06; collision box size=0.18 0.020 0.06
- added link link_05_red; collision box size=0.0015 0.1 0.078; collision box size=0.0015 0.1 0.078
- link link_01: geometry collision box size=0.173 0.148 0.106; collision cylinder length=0.032 radius=0.047
- link link_02: geometry collision box size=0.006 0.28 0.076; collision box size=0.006 0.28 0.076
- link link_03: geometry collision box size=0.120 0.090 0.08; collision cylinder length=0.104 radius=0.019
- link link_04: geometry collision box size=0.06 0.006 0.18; collision box size=0.06 0.006 0.18
- link link_05: geometry collision box size=0.055 0.007 0.078; collision box size=0.055 0.1 0.007
- link link_06: geometry collision cylinder length=0.005 radius=0.024; collision cylinder length=0.0168 radius=0.0095
Joints:
- added joint link_01__link_01_red: type fixed, parent link_01, child link_01_red, origin xyz=0.01 0 0 rpy=0 0 0
- added joint link_02__link_02_red: type fixed, parent link_02, child link_02_red, origin xyz=0 0.181 0 rpy=0 0 0
- added joint link_03__link_03_red: type fixed, parent link_03, child link_03_red, origin xyz=0.04 0 0 rpy=0 0 0
- added joint link_04__link_04_red: type fixed, parent link_04, child link_04_red, origin xyz=0 0 0.181 rpy=0 0 0
- added joint link_05__link_05_red: type fixed, parent link_05, child link_05_red, origin xyz=0 0.05 0 rpy=0 0 0
- joint link_01__link_02: limit lower=-3.57 upper=0 effort=1000.0 velocity=0.5 -> lower=-3.57 upper=0.05 effort=1000.0 velocity=0.5
- joint link_02__link_03: limit lower=0.035 upper=5.23 effort=1000.0 velocity=0.5 -> lower=-0.035 upper=5.23 effort=1000.0 velocity=0.5

File: config/ruka_gz.urdf.xacro (robot description, xacro)
@@ -2,9 +2,9 @@
 <robot xmlns:xacro="http://www.ros.org/wiki/xacro" name="ruka_gz">
     <!-- <xacro:arg name="prefix" default="" /> -->
-    <!-- <xacro:arg name="initial_positions_file" default="initial_positions.yaml" /> -->
+     <!-- <xacro:arg name="initial_positions_file" default="initial_positions.yaml" />  -->
     <!-- Import ruka_hand urdf file -->
     <xacro:include filename="$(find ruka_gz)/config/ruka_gz.urdf" />
     <!-- Import control_xacro -->
     <xacro:include filename="$(find ruka_gz)/config/ruka_gz.ros2_control.xacro" />
-    <!-- <xacro:ruka_gz_ros2_control name="RukaGazeboSimSystem" initial_positions_file="$(arg initial_positions_file)"/> -->
+    <!-- <xacro:ruka_gz_ros2_control name="RukaGazeboSimSystem" initial_positions_file="$(arg initial_positions_file)"/>  -->
 </robot>

Commit message: color fixed, use_sim_time true fixed

File: config/ruka_gz.urdf (robot description, URDF)
Before this commit: robot ruka_gz, 13 links, 12 joints
Links:
- link base_link: mass 2.92 -> 2.0
- link link_01: mass 2.74 -> 2.0
- link link_02: mass 2.74 -> 1.5
- link link_03: mass 2.38 -> 1.0
- link link_04: mass 2.38 -> 0.9
- link link_05: mass 2.74 -> 0.7
- link link_06: mass 1.55 -> 0.5

Commit message: Replace world with rover_base

File: config/ruka_gz.urdf (robot description, URDF)
Before this commit: robot ruka_gz, 13 links, 12 joints
Links:
- removed link world
Joints:
- removed joint ruka_joint_world

Commit message: stable

File: config/ruka_gz.urdf (robot description, URDF)
Before this commit: robot ruka_gz, 16 links, 15 joints
Links:
- link link_hand_cyl: geometry collision mesh filename=file://$(find ruka_gz)/config/mesh/gripper4310.stl; visual mesh filename=file://$(find ruka_gz)/config/mesh/gripper4310.stl
Joints:
- joint link_hand_cyl__first_fin: limit lower=0.0 upper=0.01 effort=20 velocity=0.2 -> lower=-0.00001 upper=0.01 effort=20 velocity=0.2
- joint link_hand_cyl__second_fin: limit lower=0.0 upper=0.01 effort=20 velocity=0.2 -> lower=-0.00001 upper=0.01 effort=20 velocity=0.2
